File: pcb/ver3.1/hackaBLE.kicad_pcb (KiCad board)
At the start: 2 copper layers, 30.1 x 29.9 mm, 33 parts, among them J1 GPIO, J2 GPIO, J3 GPIO, J4 Conn_01x02_Pin, J5 GPIO, J7 SWD, SW1 SW_Push, U1 nrf52832, U3 RF_Antenna, Y1 32.768KHz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

Commit message: all is left now is to get a place for the Buzzer in the schematics.
Parts:
- added BZ1: Buzzer, Buzzer_Beeper:Buzzer_Murata_PKMCS0909E, F.Cu at (154.6, 119.0)
- moved C4 0.90 mm to (168.3, 128.1)
- moved C3 0.65 mm to (168.6, 123.4)
- moved Y1 0.30 mm to (173.1, 125.2)
Routing:
- net GND: track 64.9 -> 42.5 mm
- net /P0.14: track 9.47 -> 8.48 mm
- net /P0.13: track 10.3 -> 9.35 mm
- net /P0.10: track 30.9 -> 31.8 mm
- net /P0.09: track 31.9 -> 31.3 mm
- net /P0.03: track 22.2 -> 22.4 mm, vias 2 -> 1

Commit message: I guess that is it.. I will manufacture this for testing.
Parts:
- BZ1: footprint Buzzer_Beeper:Buzzer_Murata_PKMCS0909E -> Buzzer:BUZ-SMD_L5.0-W5.5-P4.60
- J4: value Conn_01x02_Pin -> Battery_CR2032
- moved BZ1 13.1 mm to (167.7, 118.8)
Routing:
- net VDD: track 64.5 -> 66.1 mm
- net /P0.02: track 25.8 -> 24.9 mm
- net GND: track 42.5 -> 42.7 mm, vias 33 -> 34
Other:
- board text added: "U3 design v3.1"
- board text removed: "V 3.0"

Commit message: fix: small modifications for fabrication.
Parts:
- D1: value LED_ARGB -> SX 0606 RGB LED_ARGB
- L3: value 3.9uH -> 3.9nH
Routing:
- net Net-(D1-BK): track 5.63 -> 2.43 mm
- net VDD: track 66.1 -> 63.8 mm
- net Net-(D1-GK): track 7.57 -> 5.24 mm
- net Net-(D1-RK): track 3.23 -> 4.67 mm
- net /RESET: track 32.0 -> 32.8 mm
