File: pcb/ver3.1/hackaBLE.kicad_sch (KiCad schematic)
At the start: 33 parts, among them J1 GPIO, J2 GPIO, J3 GPIO, J4 Conn_01x02_Pin, J5 GPIO, J7 SWD, SW1 SW_Push, U1 nrf52832, U3 RF_Antenna, Y1 32.768KHz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

Commit message: all is left now is to get a place for the Buzzer in the schematics.
Parts:
- added BZ1: Buzzer, Buzzer_Beeper:Buzzer_Murata_PKMCS0909E, symbol Device:Buzzer
- J4: footprint (none) -> Battery:BatteryHolder_MYOUNG_BS-07-A1BJ001_CR2032
Connections:
- net GND: now also BZ1.2 (-)
- net P0.02: now also BZ1.1 (+)
Changed lines of the file:
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@@
 		(title "hackaBLE")
 		(date "2025-08-06")
-		(rev "Ver 3.0")
+		(rev "Ver 3.1")
 		(company "electronut Labs")
 		(comment 1 "Edit by Mohamed U3")
@@
 	(wire
 		(pts
+			(xy 231.14 74.93) (xy 236.22 74.93)
+		)
+		(stroke
+			(width 0)
+			(type default)
+		)
+	)
+	(wire
+		(pts
 			(xy 53.34 116.84) (xy 60.96 116.84)
 		)
@@
 	(wire
 		(pts
+			(xy 233.68 80.01) (xy 236.22 80.01)
+		)
+		(stroke
+			(width 0)
+			(type default)
+		)
+	)
+	(wire
+		(pts
 			(xy 86.36 83.82) (xy 86.36 87.63)
 		)
@@
 		)
 	)
+	(label "P0.02"
+		(at 231.14 74.93 0)
+		(effects
+			(font
+				(size 0.9906 0.9906)
+			)
+			(justify left bottom)
+		)
+	)
 	(label "P0.08"
 		(at 53.34 127 0)
@@
 		(lib_name "GND_21")
 		(lib_id "hackaBLE-rescue:GND")
+		(at 233.68 80.01 270)
+		(unit 1)
+		(exclude_from_sim no)
+		(in_bom yes)
+		(on_board yes)
+		(dnp no)
+		(property "Reference" "#PWR024"
+			(at 227.33 80.01 0)
+			(effects
+				(font
+					(size 1.27 1.27)
+				)
+				(hide yes)
+			)
+		)
+		(property "Value" "GND"
+			(at 229.87 80.01 0)
+			(effects
+				(font
+					(size 1.27 1.27)
+				)
+			)
+		)
+		(property "Footprint" ""
+			(at 233.68 80.01 0)
+			(effects
+				(font
+					(size 1.27 1.27)
+				)
+				(hide yes)
+			)
+		)
+		(property "Datasheet" ""
+			(at 233.68 80.01 0)
+			(effects
+				(font
+					(size 1.27 1.27)
+				)
+				(hide yes)
+			)
+		)
+		(property "Description" ""
+			(at 233.68 80.01 0)
+			(effects
+				(font
+					(size 1.27 1.27)
+				)
+			)
+		)
+		(pin "1"
+		)
+		(instances
+			(project "hackaBLE"
+				(path "/7bf155d7-cf3f-4b19-a6e4-e06ff318c707"
+					(reference "#PWR024")
+					(unit 1)
+				)
+			)
+		)
+	)
+	(symbol
+		(lib_name "GND_21")
+		(lib_id "hackaBLE-rescue:GND")
 		(at 246.38 35.56 90)
 		(unit 1)
@@
 	)
 	(symbol
+		(lib_id "Device:Buzzer")
+		(at 238.76 77.47 0)
+		(unit 1)
+		(exclude_from_sim no)
+		(in_bom yes)
+		(on_board yes)
+		(dnp no)
+		(fields_autoplaced yes)
+		(property "Reference" "BZ1"
+			(at 242.57 76.1999 0)
+			(effects
+				(font
+					(size 1.27 1.27)
+				)
+				(justify left)
+			)
+		)
+		(property "Value" "Buzzer"
+			(at 242.57 78.7399 0)
+			(effects
+				(font
+					(size 1.27 1.27)
+				)
+				(justify left)
+			)
+		)
+		(property "Footprint" "Buzzer_Beeper:Buzzer_Murata_PKMCS0909E"
+			(at 238.125 74.93 90)
+			(effects
+				(font
+					(size 1.27 1.27)
+				)
+				(hide yes)
+			)
+		)
+		(property "Datasheet" "~"
+			(at 238.125 74.93 90)
+			(effects
+				(font
+					(size 1.27 1.27)
+				)
+				(hide yes)
+			)
+		)
+		(property "Description" "Buzzer, polarized"
+			(at 238.76 77.47 0)
+			(effects
+				(font
+					(size 1.27 1.27)
+				)
+				(hide yes)
+			)
+		)
+		(pin "1"
+		)
+		(pin "2"
+		)
+		(instances
+			(project ""
+				(path "/7bf155d7-cf3f-4b19-a6e4-e06ff318c707"
+					(reference "BZ1")
+					(unit 1)
+				)
+			)
+		)
+	)
+	(symbol
 		(lib_id "Connector:Conn_01x02_Pin")
 		(at 234.95 35.56 0)
@@
 			)
 		)
-		(property "Footprint" ""
+		(property "Footprint" "Battery:BatteryHolder_MYOUNG_BS-07-A1BJ001_CR2032"
 			(at 234.95 35.56 0)
 			(effects

Commit message: I guess that is it.. I will manufacture this for testing.
Parts:
- BZ1: footprint Buzzer_Beeper:Buzzer_Murata_PKMCS0909E -> Buzzer:BUZ-SMD_L5.0-W5.5-P4.60
- J4: value Conn_01x02_Pin -> Battery_CR2032
Other:
- moved on the sheet: BZ1, J4
Changed lines of the file:
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@@
 	(rectangle
 		(start 43.19 12.57)
-		(end 143.45 59.83)
+		(end 143.45 59.69)
 		(stroke
 			(width 0.508)
@@
 	(rectangle
 		(start 12.85 12.52)
-		(end 42.6 59.86)
+		(end 42.6 59.69)
 		(stroke
 			(width 0.508)
@@
 	(wire
 		(pts
-			(xy 240.03 38.1) (xy 243.84 38.1)
+			(xy 222.25 31.75) (xy 226.06 31.75)
 		)
 		(stroke
@@
 	(wire
 		(pts
-			(xy 243.84 39.37) (xy 246.38 39.37)
+			(xy 226.06 33.02) (xy 228.6 33.02)
 		)
 		(stroke
@@
 	(wire
 		(pts
-			(xy 231.14 74.93) (xy 236.22 74.93)
+			(xy 257.81 27.94) (xy 262.89 27.94)
 		)
 		(stroke
@@
 	(wire
 		(pts
-			(xy 243.84 38.1) (xy 243.84 39.37)
+			(xy 226.06 31.75) (xy 226.06 33.02)
 		)
 		(stroke
@@
 	(wire
 		(pts
-			(xy 240.03 35.56) (xy 246.38 35.56)
+			(xy 222.25 29.21) (xy 228.6 29.21)
 		)
 		(stroke
@@
 	(wire
 		(pts
-			(xy 233.68 80.01) (xy 236.22 80.01)
+			(xy 260.35 33.02) (xy 262.89 33.02)
 		)
 		(stroke
@@
 	)
 	(label "P0.02"
-		(at 231.14 74.93 0)
+		(at 257.81 27.94 0)
 		(effects
 			(font
@@
 		(lib_name "GND_21")
 		(lib_id "hackaBLE-rescue:GND")
-		(at 233.68 80.01 270)
+		(at 260.35 33.02 270)
 		(unit 1)
 		(exclude_from_sim no)
@@
 		(dnp no)
 		(property "Reference" "#PWR024"
-			(at 227.33 80.01 0)
+			(at 254 33.02 0)
 			(effects
 				(font
@@
 		)
 		(property "Value" "GND"
-			(at 229.87 80.01 0)
+			(at 256.54 33.02 0)
 			(effects
 				(font
@@
 		)
 		(property "Footprint" ""
-			(at 233.68 80.01 0)
+			(at 260.35 33.02 0)
 			(effects
 				(font
@@
 		)
 		(property "Datasheet" ""
-			(at 233.68 80.01 0)
+			(at 260.35 33.02 0)
 			(effects
 				(font
@@
 		)
 		(property "Description" ""
-			(at 233.68 80.01 0)
+			(at 260.35 33.02 0)
 			(effects
 				(font
@@
 		(lib_name "GND_21")
 		(lib_id "hackaBLE-rescue:GND")
-		(at 246.38 35.56 90)
+		(at 228.6 29.21 90)
 		(unit 1)
 		(exclude_from_sim no)
@@
 		(dnp no)
 		(property "Reference" "#PWR022"
-			(at 252.73 35.56 0)
+			(at 234.95 29.21 0)
 			(effects
 				(font
@@
 		)
 		(property "Value" "GND"
-			(at 250.19 35.56 0)
+			(at 232.41 29.21 0)
 			(effects
 				(font
@@
 		)
 		(property "Footprint" ""
-			(at 246.38 35.56 0)
+			(at 228.6 29.21 0)
 			(effects
 				(font
@@
 		)
 		(property "Datasheet" ""
-			(at 246.38 35.56 0)
+			(at 228.6 29.21 0)
 			(effects
 				(font
@@
 		)
 		(property "Description" ""
-			(at 246.38 35.56 0)
+			(at 228.6 29.21 0)
 			(effects
 				(font
@@
 	(symbol
 		(lib_id "Device:Buzzer")
-		(at 238.76 77.47 0)
+		(at 265.43 30.48 0)
 		(unit 1)
 		(exclude_from_sim no)
@@
 		(fields_autoplaced yes)
 		(property "Reference" "BZ1"
-			(at 242.57 76.1999 0)
+			(at 269.24 29.2099 0)
 			(effects
 				(font
@@
 		)
 		(property "Value" "Buzzer"
-			(at 242.57 78.7399 0)
+			(at 269.24 31.7499 0)
 			(effects
 				(font
@@
 			)
 		)
-		(property "Footprint" "Buzzer_Beeper:Buzzer_Murata_PKMCS0909E"
-			(at 238.125 74.93 90)
+		(property "Footprint" "Buzzer:BUZ-SMD_L5.0-W5.5-P4.60"
+			(at 264.795 27.94 90)
 			(effects
 				(font
@@
 		)
 		(property "Datasheet" "~"
-			(at 238.125 74.93 90)
+			(at 264.795 27.94 90)
 			(effects
 				(font
@@
 		)
 		(property "Description" "Buzzer, polarized"
-			(at 238.76 77.47 0)
+			(at 265.43 30.48 0)
 			(effects
 				(font
@@
 	(symbol
 		(lib_id "Connector:Conn_01x02_Pin")
-		(at 234.95 35.56 0)
+		(at 217.17 29.21 0)
 		(unit 1)
 		(exclude_from_sim no)
@@
 		(fields_autoplaced yes)
 		(property "Reference" "J4"
-			(at 235.585 30.48 0)
+			(at 217.805 24.13 0)
 			(effects
 				(font
@@
 			)
 		)
-		(property "Value" "Conn_01x02_Pin"
-			(at 235.585 33.02 0)
+		(property "Value" "Battery_CR2032"
+			(at 217.805 26.67 0)
 			(effects
 				(font
@@
 		)
 		(property "Footprint" "Battery:BatteryHolder_MYOUNG_BS-07-A1BJ001_CR2032"
-			(at 234.95 35.56 0)
+			(at 217.17 29.21 0)
 			(effects
 				(font
@@
 		)
 		(property "Datasheet" "~"
-			(at 234.95 35.56 0)
+			(at 217.17 29.21 0)
 			(effects
 				(font
@@
 		)
 		(property "Description" "Generic connector, single row, 01x02, script generated"
-			(at 234.95 35.56 0)
+			(at 217.17 29.21 0)
 			(effects
 				(font
@@
 		(lib_name "VDD_9")
 		(lib_id "hackaBLE-rescue:VDD")
-		(at 246.38 39.37 270)
+		(at 228.6 33.02 270)
 		(unit 1)
 		(exclude_from_sim no)
@@
 		(dnp no)
 		(property "Reference" "#PWR023"
-			(at 242.57 39.37 0)
+			(at 224.79 33.02 0)
 			(effects
 				(font
@@
 		)
 		(property "Value" "VDD"
-			(at 250.19 39.37 0)
+			(at 232.41 33.02 0)
 			(effects
 				(font
@@
 		)
 		(property "Footprint" ""
-			(at 246.38 39.37 0)
+			(at 228.6 33.02 0)
 			(effects
 				(font
@@
 		)
 		(property "Datasheet" ""
-			(at 246.38 39.37 0)
+			(at 228.6 33.02 0)
 			(effects
 				(font
@@
 		)
 		(property "Description" ""
-			(at 246.38 39.37 0)
+			(at 228.6 33.02 0)
 			(effects
 				(font

Commit message: fix: small modifications for fabrication.
Parts:
- D1: value LED_ARGB -> SX 0606 RGB LED_ARGB
- L3: value 3.9uH -> 3.9nH
Changed lines of the file:
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@@
 			)
 		)
-		(property "Value" "LED_ARGB"
+		(property "Value" "SX 0606 RGB LED_ARGB"
 			(at 167.64 27.94 0)
 			(effects
@@
 			)
 		)
-		(property "Description" ""
-			(at 167.64 36.83 0)
-			(effects
-				(font
-					(size 1.27 1.27)
-				)
+		(property "Description" "SX 0606 RGB"
+			(at 157.48 38.862 0)
+			(effects
+				(font
+					(size 1.27 1.27)
+				)
+				(hide yes)
 			)
 		)
@@
 			)
 		)
-		(property "Value" "3.9uH"
+		(property "Value" "3.9nH"
 			(at 156.972 120.523 90)
 			(effects
@@
 			)
 		)
-		(property "Description" ""
+		(property "Description" "LQP15MN3N9B02D"
 			(at 154.94 119.38 0)
 			(effects
@@
 					(size 1.27 1.27)
 				)
-			)
-		)
+				(hide yes)
+			)
+		)
